Commit message: Update vg10 collision boundary

File: urdf/vg10.xacro (robot description, xacro)
@@ -3,61 +3,47 @@
   <link name="vg10_quick_changer">
     <visual>
-      <origin xyz="0 0 0" rpy="${-pi/2} 0 ${-pi/2}"/>
+      <origin xyz="0 0 0" rpy="${-pi/2} 0 ${-pi/2}" />
       <geometry>
-        <mesh filename="package://ros2_vg10_gripper/meshes/quick_changer.stl" scale="0.001 0.001 0.001"/>
+        <mesh filename="package://ros2_vg10_gripper/meshes/quick_changer.stl"
+          scale="0.001 0.001 0.001" />
       </geometry>
       <material name="blue">
-        <color rgba="0.196078431 0.462745098 0.560784314 1.0"/>
+        <color rgba="0.196078431 0.462745098 0.560784314 1.0" />
       </material>
     </visual>
     <!-- In practice, this mounting bracket will never collide with anything.  -->
     <!-- <collision> -->
-      <!-- TODO(elvout): This could probably be a cylinder to reduce computational load. -->
-      <!-- <origin xyz="0 0 0" rpy="${-pi/2} 0 ${-pi/2}" /> -->
-      <!-- <geometry> -->
-        <!-- <mesh filename="package://neo_mpo_700-2/robot_model/meshes/vg10_quick_changer.stl" scale="0.001 0.001 0.001"/> -->
-      <!-- </geometry> -->
+    <!-- TODO(elvout): This could probably be a cylinder to reduce computational load. -->
+    <!-- <origin xyz="0 0 0" rpy="${-pi/2} 0 ${-pi/2}" /> -->
+    <!-- <geometry> -->
+    <!-- <mesh filename="package://neo_mpo_700-2/robot_model/meshes/vg10_quick_changer.stl"
+    scale="0.001 0.001 0.001"/> -->
+    <!-- </geometry> -->
     <!-- </collision> -->
   </link>
   <link name="vg10">
     <visual>
-      <origin xyz="0 0 0" rpy="${-pi/2} 0 ${-pi/2}"/>
+      <origin xyz="0 0 0" rpy="${-pi/2} 0 ${-pi/2}" />
       <geometry>
-        <mesh filename="package://ros2_vg10_gripper/meshes/vg10.stl" scale="0.001 0.001 0.001"/>
+        <mesh filename="package://ros2_vg10_gripper/meshes/vg10.stl" scale="0.001 0.001 0.001" />
       </geometry>
       <material name="gray">
-        <color rgba="0.5 0.5 0.5 1.0"/>
+        <color rgba="0.5 0.5 0.5 1.0" />
       </material>
     </visual>
     <collision>
-      <!-- TODO(elvout): This could probably be a cube to reduce computational load. -->
-      <origin xyz="0 0 0" rpy="${-pi/2} 0 ${-pi/2}" />
+      <!-- <origin xyz="0 0 0" rpy="${-pi/2} 0 ${-pi/2}" />
       <geometry>
         <mesh filename="package://ros2_vg10_gripper/meshes/vg10.stl" scale="0.001 0.001 0.001"/>
-      </geometry>
-    </collision>
-  </link>
-  <!--
-    TODO(elvout) merge into vg10 collision property with a warning to visually
-    check the bounding box using the visual parameter when making any changes.
-    Using a bounding box instead of a convex hull because (a) it has simpler
-    geometry and (b) the tolerance of the rounded edges is very low and the
-    precision required to avoid a collision is very high. The corners of the
-    simpler box add some safety buffer.
-  -->
-  <link name="vg10_bbox">
-    <visual>
-      <origin xyz="0 0 ${0.09 / 2 + 0.12 - 0.09}" rpy="0 0 0"/>
-      <geometry>
-        <!-- True size is X Y Z 0.146 0.146 0.1186. -->
-        <box size="0.146 0.146 0.09"/>
-      </geometry>
-      <material name="gray">
-        <color rgba="0.5 0.5 0.5 0.25" />
-      </material>
-    </visual>
-    <collision>
+      </geometry> -->
+      <!-- IMPORTANT: ALWAYS VERIFY COLLISION BOUNDARY IN RVIZ -->
+      <!--
+      Using a bounding box because the tolerance of the gripper's rounded edges
+      are very small. The precision required to avoid a collision is very high.
+      The corners of the box add some safety buffer space. Could be made more
+      precise with a convex hull with some safety margin.
+      -->
+      <!-- True z-length is 0.1186 -->
       <origin xyz="0 0 ${0.09 / 2 + 0.12 - 0.09}" rpy="0 0 0" />
-      <!-- TODO(elvout): This could probably be a cube to reduce computational load. -->
       <geometry>
         <box size="0.146 0.146 0.09" />
@@ -65,5 +51,5 @@
     </collision>
   </link>
-  <link name="vg10_grasp_center"/>
+  <link name="vg10_grasp_center" />
   <joint name="vg10_quick_changer_joint" type="fixed">
     <parent link="$(arg tf_prefix)tool0" />
@@ -77,14 +63,9 @@
     <origin xyz="0 0 0" rpy="0 0 0" />
   </joint>
-  <joint name="vg10_bbox_mount_joint" type="fixed">
-    <parent link="vg10_quick_changer" />
-    <child link="vg10_bbox" />
-    <origin xyz="0 0 0" rpy="0 0 0" />
-  </joint>
   <joint name="vg10_grasp_center_joint" type="fixed">
-      <parent link="vg10"/>
-      <child link="vg10_grasp_center"/>
-      <!-- Derived from gripper + quick changer datasheets. -->
-      <origin xyz="0 0 0.1186" rpy="0 0 0"/>
+    <parent link="vg10" />
+    <child link="vg10_grasp_center" />
+    <!-- Derived from gripper + quick changer datasheets. -->
+    <origin xyz="0 0 0.1186" rpy="0 0 0" />
   </joint>
 </robot>
